Commit message: Acrobot controller

File: acrobot_simulator/acrobot_description/urdf/acrobot.xacro (robot description, xacro)
@@ -72,5 +72,5 @@
     <origin xyz="0 0 0.3" rpy="${PI/2} 0 0"/>
     <axis xyz="0 1 0"/>
-    <dynamics damping="0.1"/>
+    <!-- <dynamics damping="0.1"/> -->
   </joint>
   <joint name="joint2" type="continuous">

Commit message: Vertical configuration

File: acrobot_simulator/acrobot_description/urdf/acrobot.xacro (robot description, xacro)
@@ -70,5 +70,6 @@
     <parent link="world"/>
     <child link="link1"/>
-    <origin xyz="0 0 0.3" rpy="${PI/2} 0 0"/>
+    <origin xyz="0 0 ${height1 + height2 + axel_offset2}" rpy="0 ${PI} 0"/>
+    <!-- <origin xyz="0 0 0.3" rpy="${PI/2} 0 0"/> -->
     <axis xyz="0 1 0"/>
     <!-- <dynamics damping="0.1"/> -->
